File: tm9.brd (EAGLE design)
At the start: 41.9 x 41.9 mm, 42 parts, among them J1 DF23C-10DP-0.5V(92), J2 DF23C-10DP-0.5V(92), U2 ARTEMIS_MODULESMD, Y1 32.768kHz

Commit message: rough draft
added JST-SH 6-pin RA connector, 1mA battery, and just shuffled around parts to get a general feel for things. Just a very rough draft.
Parts:
- added BT2: RELOWABLE_BATTERY_ML414H, SparkFun-Batteries:ML414H_IV01E
- J3: device SparkFun-Connectors:USB-MICROB -> SparkFun-Connectors:JST-6-SMD-1.25MM-LOCKING
- moved R23 3.62 mm to (37.9, 41.4)
- moved C11 1.12 mm to (42.9, 42.9)
- moved U$1 1.12 mm to (40.6, 42.7)
- moved J1 1.11 mm to (61.1, 36.8)
- moved J3 0.57 mm to (32.1, 44.8), turned to 90 degrees
Connections:
- removed net VBUS: J3.VBUS
- net +: now also BT2.+
- net -: now also BT2.-
- net GND: no longer J3.GND
Routing:
- net XIN32: track 0.00 -> 3.99 mm
- net XOUT32: track 0.00 -> 3.16 mm

Commit message: added SCL and SDA labels
added SCL and SDA labels for all I2C ports on Artemis module.

labeled both I2C LCDs accordingly for shortest I2C trace length.
Parts:
- added U1: SST25VF020BUSON, SparkFun-IC-Memory:USON_3X2MM
Connections:
- new net SCL0: U2.~D5
- new net SCL2: LCD1.4, R1.1, U2.~D27
- new net SCL3: U2.~D42
- new net SCL4: U2.~D39
- new net SDA0: U2.~D6
- new net SDA2: LCD1.5, R2.1, U2.~D25
- new net SDA3: U2.~D43
- new net SDA4: U2.D40
- new net VCC: U1.8
- net GND: now also U1.4
- net SCL: no longer LCD1.4, R1.1
- net SCL1: now also U2.D8
- net SDA: no longer LCD1.5, R2.1
- net SDA1: now also U2.D9
Changed lines of the file:
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@@
 <attribute name="VALUE" x="54.70525" y="40.132" size="0.381" layer="28" rot="MR180"/>
+</element>
+<element name="U1" library="SparkFun-IC-Memory" package="USON_3X2MM" value="SST25VF020BUSON" x="47.3075" y="43.65625" smashed="yes" rot="MR270">
+<attribute name="DIGIKEY_PART" value="SST25VF020B-80-4I-Q3AE-TCT-ND" x="47.3075" y="43.65625" size="1.778" layer="28" rot="MR270" display="off"/>
+<attribute name="MANU_PART" value="SST25VF020B-80-4I-Q3AE-T" x="47.3075" y="43.65625" size="1.778" layer="28" rot="MR270" display="off"/>
+<attribute name="PROD_ID" value="IC-15716" x="47.3075" y="43.65625" size="1.778" layer="28" rot="MR270" display="off"/>
+<attribute name="VALUE" x="49.3075" y="43.65625" size="0.6096" layer="28" font="vector" ratio="20" rot="MR270" align="bottom-center"/>
 </element>
 </elements>
@@
 <contactref element="U$1" pad="P$6"/>
 <contactref element="LS1" pad="P"/>
-<wire x1="51.1175" y1="37.5275" x2="65.65176875" y2="46.5338875" width="0" layer="19" extent="1-1"/>
-<wire x1="48.5775" y1="37.5275" x2="51.1175" y2="37.5275" width="0" layer="19" extent="1-1"/>
-<wire x1="46.125" y1="34.29" x2="48.5775" y2="37.5275" width="0" layer="19" extent="1-1"/>
-<wire x1="44.1325" y1="28.575" x2="46.125" y2="34.29" width="0" layer="19" extent="1-1"/>
+<contactref element="U1" pad="4"/>
+<wire x1="48.0575" y1="44.98125" x2="65.65176875" y2="46.5338875" width="0" layer="19" extent="1-16"/>
+<wire x1="66.04" y1="26.44" x2="48.0575" y2="44.98125" width="0" layer="19" extent="16-16"/>
+<wire x1="65.65176875" y1="25.856109375" x2="66.04" y2="26.44" width="0" layer="19" extent="1-16"/>
+<wire x1="63.5" y1="23.18875" x2="65.65176875" y2="25.856109375" width="0" layer="19" extent="1-16"/>
+<wire x1="54.06198125" y1="26.81625" x2="63.5" y2="23.18875" width="0" layer="19" extent="1-16"/>
+<wire x1="51.1175" y1="28.575" x2="54.06198125" y2="26.81625" width="0" layer="19" extent="1-1"/>
+<wire x1="54.06198125" y1="30.33375" x2="51.1175" y2="28.575" width="0" layer="19" extent="1-1"/>
+<wire x1="44.1325" y1="28.575" x2="51.1175" y2="28.575" width="0" layer="19" extent="1-1"/>
 <wire x1="41.188015625" y1="30.33375" x2="44.1325" y2="28.575" width="0" layer="19" extent="1-1"/>
 <wire x1="41.188015625" y1="26.81625" x2="44.1325" y2="28.575" width="0" layer="19" extent="1-1"/>
-<wire x1="51.1175" y1="28.575" x2="44.1325" y2="28.575" width="0" layer="19" extent="1-1"/>
-<wire x1="54.06198125" y1="30.33375" x2="51.1175" y2="28.575" width="0" layer="19" extent="1-1"/>
-<wire x1="54.06198125" y1="26.81625" x2="51.1175" y2="28.575" width="0" layer="19" extent="1-1"/>
-<wire x1="39.0525" y1="37.5275" x2="41.188015625" y2="30.33375" width="0" layer="19" extent="1-1"/>
+<wire x1="46.125" y1="34.29" x2="44.1325" y2="28.575" width="0" layer="19" extent="1-1"/>
+<wire x1="48.5775" y1="37.5275" x2="46.125" y2="34.29" width="0" layer="19" extent="1-1"/>
+<wire x1="51.1175" y1="37.5275" x2="48.5775" y2="37.5275" width="0" layer="19" extent="1-1"/>
+<wire x1="42.8625" y1="42.2125" x2="48.5775" y2="37.5275" width="0" layer="19" extent="1-16"/>
+<wire x1="41.63" y1="41.95375" x2="42.8625" y2="42.2125" width="0" layer="19" extent="16-16"/>
+<wire x1="40.64" y1="42.70375" x2="41.63" y2="41.95375" width="0" layer="19" extent="16-16"/>
+<wire x1="39.65" y1="42.45375" x2="40.64" y2="42.70375" width="0" layer="19" extent="16-16"/>
+<wire x1="41.63" y1="43.45375" x2="40.64" y2="42.70375" width="0" layer="19" extent="16-16"/>
+<wire x1="39.0525" y1="37.5275" x2="39.65" y2="42.45375" width="0" layer="19" extent="1-16"/>
 <wire x1="36.5125" y1="37.5275" x2="39.0525" y2="37.5275" width="0" layer="19" extent="1-1"/>
-<wire x1="39.65" y1="42.45375" x2="39.0525" y2="37.5275" width="0" layer="19" extent="1-16"/>
-<wire x1="40.64" y1="42.70375" x2="39.65" y2="42.45375" width="0" layer="19" extent="16-16"/>
-<wire x1="41.63" y1="43.45375" x2="40.64" y2="42.70375" width="0" layer="19" extent="16-16"/>
-<wire x1="41.63" y1="41.95375" x2="40.64" y2="42.70375" width="0" layer="19" extent="16-16"/>
-<wire x1="42.8625" y1="42.2125" x2="41.63" y2="41.95375" width="0" layer="19" extent="16-16"/>
 <wire x1="46.19625" y1="47.79875" x2="41.63" y2="43.45375" width="0" layer="19" extent="16-16"/>
 <wire x1="46.19625" y1="48.72125" x2="46.19625" y2="47.79875" width="0" layer="19" extent="16-16"/>
-<wire x1="63.5" y1="23.18875" x2="54.06198125" y2="26.81625" width="0" layer="19" extent="1-16"/>
-<wire x1="65.65176875" y1="25.856109375" x2="63.5" y2="23.18875" width="0" layer="19" extent="1-16"/>
-<wire x1="66.04" y1="26.44" x2="65.65176875" y2="25.856109375" width="0" layer="19" extent="1-16"/>
 <wire x1="29.598228125" y1="46.5338875" x2="39.65" y2="42.45375" width="0" layer="19" extent="1-16"/>
 <wire x1="29.598228125" y1="25.856109375" x2="41.188015625" y2="26.81625" width="0" layer="19" extent="1-1"/>
@@
 </signal>
 <signal name="SCL">
-<contactref element="LCD1" pad="4"/>
-<contactref element="R1" pad="1"/>
 <contactref element="R20" pad="2"/>
 <contactref element="U$1" pad="P$7"/>
-<wire x1="44.1325" y1="37.5295" x2="44.142025" y2="40.1908" width="0" layer="19" extent="1-1"/>
-<wire x1="39.65" y1="42.95375" x2="44.142025" y2="40.1908" width="0" layer="19" extent="1-16"/>
-<wire x1="38.57625" y1="43.52125" x2="39.65" y2="42.95375" width="0" layer="19" extent="16-16"/>
+<wire x1="39.65" y1="42.95375" x2="38.57625" y2="43.52125" width="0" layer="19" extent="16-16"/>
 </signal>
 <signal name="SDA">
-<contactref element="LCD1" pad="5"/>
-<contactref element="R2" pad="1"/>
 <contactref element="R21" pad="2"/>
 <contactref element="U$1" pad="P$8"/>
-<wire x1="46.6725" y1="37.5275" x2="46.326425" y2="40.1908" width="0" layer="19" extent="1-1"/>
-<wire x1="39.65" y1="43.45375" x2="46.326425" y2="40.1908" width="0" layer="19" extent="1-16"/>
 <wire x1="37.465" y1="43.52125" x2="39.65" y2="43.45375" width="0" layer="19" extent="16-16"/>
 </signal>
@@
 <contactref element="LCD2" pad="5"/>
 <contactref element="R15" pad="1"/>
-<wire x1="58.01995" y1="40.04475" x2="58.7375" y2="37.5275" width="0" layer="19" extent="1-1"/>
+<contactref element="U2" pad="D9"/>
+<wire x1="58.01995" y1="40.04475" x2="58.515" y2="41.385" width="0" layer="19" extent="1-16"/>
+<wire x1="58.7375" y1="37.5275" x2="58.01995" y2="40.04475" width="0" layer="19" extent="1-1"/>
 </signal>
 <signal name="SCL1">
 <contactref element="LCD2" pad="4"/>
 <contactref element="R16" pad="1"/>
+<contactref element="U2" pad="D8"/>
+<wire x1="56.015" y1="40.585" x2="55.93715" y2="40.04475" width="0" layer="19" extent="1-16"/>
 <wire x1="56.1975" y1="37.5295" x2="55.93715" y2="40.04475" width="0" layer="19" extent="1-1"/>
 </signal>
@@
 <wire x1="57.74325" y1="34.798" x2="53.545" y2="32.50625" width="0" layer="19" extent="16-16"/>
 </signal>
+<signal name="SCL0">
+<contactref element="U2" pad="~D5"/>
+</signal>
+<signal name="SDA0">
+<contactref element="U2" pad="~D6"/>
+</signal>
+<signal name="SDA2">
+<contactref element="U2" pad="~D25"/>
+<contactref element="LCD1" pad="5"/>
+<contactref element="R2" pad="1"/>
+<wire x1="50.015" y1="42.585" x2="46.326425" y2="40.1908" width="0" layer="19" extent="1-16"/>
+<wire x1="46.6725" y1="37.5275" x2="46.326425" y2="40.1908" width="0" layer="19" extent="1-1"/>
+</signal>
+<signal name="SCL2">
+<contactref element="U2" pad="~D27"/>
+<contactref element="LCD1" pad="4"/>
+<contactref element="R1" pad="1"/>
+<wire x1="44.142025" y1="40.1908" x2="52.015" y2="40.585" width="0" layer="19" extent="1-16"/>
+<wire x1="44.1325" y1="37.5295" x2="44.142025" y2="40.1908" width="0" layer="19" extent="1-1"/>
+</signal>
+<signal name="SCL4">
+<contactref element="U2" pad="~D39"/>
+</signal>
+<signal name="SDA4">
+<contactref element="U2" pad="D40"/>
+</signal>
+<signal name="SCL3">
+<contactref element="U2" pad="~D42"/>
+</signal>
+<signal name="SDA3">
+<contactref element="U2" pad="~D43"/>
+</signal>
+<signal name="VCC">
+<contactref element="U1" pad="8"/>
+</signal>
 </signals>
